File: p1/_autosave-pcb-dualdrum.sch (KiCad schematic (older format))
At the start: 130 parts

Commit message: added notes
Other:
- note added: "que hacer\n-usar LMC7660\n-usar lm13700 filtering circuit\n-usar lm13700 en VCA config\n\nel dd necesita usar +/-9V\nhace layout por la CMOS chips con dos supply circuitos\n"
Changed lines of the file:
@@
 Wire Wire Line
 	15525 1525 16250 1525
+Text Notes 6675 1950 0    100  ~ 20
+que hacer\n-usar LMC7660\n-usar lm13700 filtering circuit\n-usar lm13700 en VCA config\n\nel dd necesita usar +/-9V\nhace layout por la CMOS chips con dos supply circuitos\n
 $EndSCHEMATC
