File: p1/pcb-dualdrum.sch (KiCad schematic (older format))
At the start: 135 parts

Commit message: wip on lm13700 circuits
Parts:
- added C? (x2): 800pF, 4ms_Capacitor:C_0603, symbol 4ms-passives:C_Small
- added Freq1, Level_?: 100k, 4ms_Potentiometer:Pot_16mm_NoDet_RV16AF-4A, symbol 4ms-mech:POT
- added R?: 13k, 4ms_Resistor:R_0603, symbol 4ms-passives:R
- added R? (x3): 30k, 4ms_Resistor:R_0603, symbol 4ms-passives:R
- added R?: 5k, 4ms_Resistor:R_0603, symbol 4ms-passives:R
- added R? (x4): 1k, 4ms_Resistor:R_0603, symbol 4ms-passives:R
- added R?: 10k, 4ms_Resistor:R_0603, symbol 4ms-passives:R
- added R? (x3): 20k, 4ms_Resistor:R_0603, symbol 4ms-passives:R
- added R? (x2): 5k1, 4ms_Resistor:R_0603, symbol 4ms-passives:R
- added R?: 15k, 4ms_Resistor:R_0603, symbol 4ms-passives:R
- added U? (x7): LM13700, symbol Amplifier_Operational:LM13700
Connections:
- wire segments 261 -> 299
- no-connect marks 7 -> 10
Other:
- moved on the sheet: U?A

Commit message: wip incorperated PI circuit
Parts:
- removed C?: 20pF, 4ms_Capacitor:C_0603, symbol 4ms-passives:C_Small
- removed ENV_LED?, GATE_LED?: LED, 4ms_LED:LED_0603_1608Metric, symbol 4ms-passives:LED
- removed H?: Env Outs, 4ms_Connector:Pins_1x03_2.54mm_TH, symbol 4ms-headers:HEADER1x3
- removed H?: 1/4in Input, 4ms_Connector:Pins_1x03_2.54mm_TH, symbol 4ms-headers:HEADER1x3
- removed INL?: JACK-MONO, 4ms_Jack:EighthInch_PJ398SM, symbol 4ms-mech:JACK-MONO
- removed R? (x2): 1k, 4ms_Resistor:R_0603, symbol 4ms-passives:R
- removed R?: 47k, 4ms_Resistor:R_0603, symbol 4ms-passives:R
- removed R? (x2): 10k, 4ms_Resistor:R_0603, symbol 4ms-passives:R
- removed R? (x2): 100k, 4ms_Resistor:R_0603, symbol 4ms-passives:R
- removed R?: 1k - this value may be wrong on Proto, 4ms_Resistor:R_0603, symbol 4ms-passives:R
- removed R?: 5k - this works, 4ms_Resistor:R_0603, symbol 4ms-passives:R
- added Aux_Gain1: 100k, 4ms_Potentiometer:Pot_16mm_NoDet_RV16AF-4A, symbol 4ms-mech:POT
- added Aux_In1: JACK-MONO, 4ms_Jack:EighthInch_PJ398SM, symbol 4ms-mech:JACK-MONO
- added C? (x2): 220pF, 4ms_Capacitor:C_0603, symbol 4ms-passives:C_Small
- added C? (x2): 1uF, 4ms_Capacitor:C_0603, symbol 4ms-passives:C_Small
- added Fol_Gen_SW?: SPST, 4ms_Switch:Slide_Switch_Runrun_SS22D06, symbol 4ms-mech:DPDT-shielded-sep
- added R? (x4): 1k, 4ms_Resistor:R_0603, symbol 4ms-passives:R
- added R?: 10k, 4ms_Resistor:R_0603, symbol 4ms-passives:R
- added R?: 100k, 4ms_Resistor:R_0603, symbol 4ms-passives:R
- added R?: 100K, 4ms_Resistor:R_0603, symbol 4ms-passives:R
- added U?: NJM, 4ms_Package_SSOP:TSSOP-8_4.4x3mm_Pitch0.65mm, symbol 4ms-ic:NJM2068-separate-power
- added U? (x2): 072, 4ms_Package_SSOP:TSSOP-8_4.4x3mm_Pitch0.65mm, symbol 4ms-ic:NJM2068-separate-power
- C? (x2): value 220pF - 1000pF -> 220pF
- R?: value 220k -> 10k
- gave numbers to parts that had none: 4
Connections:
- wire segments 299 -> 309
- no-connect marks 10 -> 9
Other:
- note added: "VCA"
- moved on the sheet: C?, D?, ENV_LED?, EnvSense?, Fol_Gen_SW1A, Freq1, GATE?, H?, INL?, L?, LED?, Level_?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

Commit message: ok time to take a break
Parts:
- added C?: 200pF, 4ms_Capacitor:C_0603, symbol 4ms-passives:C_Small
- added Pitch, Slide1, Wave1: 100k, 4ms_Potentiometer:Pot_16mm_NoDet_RV16AF-4A, symbol 4ms-mech:POT
- added R? (x2): 30k, 4ms_Resistor:R_0603, symbol 4ms-passives:R
- added R? (x2): 10k, 4ms_Resistor:R_0603, symbol 4ms-passives:R
- added R?: 5k1, 4ms_Resistor:R_0603, symbol 4ms-passives:R
- added R?: 51k, 4ms_Resistor:R_0603, symbol 4ms-passives:R
- added U? (x5): LM13700, symbol Amplifier_Operational:LM13700
Connections:
- wire segments 309 -> 334
- no-connect marks 9 -> 11
Other:
- note added: "AUX GAIN"
- note added: "VCO"
- note added: "this slide thing seems a little silly\nmaybe i should look more into it\nor try it out...."
- note added: "what should i do about this pot?\nis it enough gain to boost signal?\ncan i use a fixed resistor?\ncan i use a pot on the cv input to attenuate?"
- moved on the sheet: U?E

Commit message: added new schem + notes
Parts:
- added C? (x2): 1000pF - 10nF, 4ms_Capacitor:C_0603, symbol 4ms-passives:C_Small
- added INL? (x2): JACK-MONO, 4ms_Jack:EighthInch_PJ398SM, symbol 4ms-mech:JACK-MONO
- added Level_?: 1M, 4ms_Potentiometer:Pot_16mm_NoDet_RV16AF-4A, symbol 4ms-mech:POT
- added R? (x4): 1k, 4ms_Resistor:R_0603, symbol 4ms-passives:R
- added R?: 22k, 4ms_Resistor:R_0603, symbol 4ms-passives:R
- added R? (x3): 20k, 4ms_Resistor:R_0603, symbol 4ms-passives:R
- added R?: 100k, 4ms_Resistor:R_0603, symbol 4ms-passives:R
- added R?: 10k, 4ms_Resistor:R_0603, symbol 4ms-passives:R
- added U? (x4): LM13700, symbol Amplifier_Operational:LM13700
- added U? (x3): NJM, 4ms_Package_SSOP:TSSOP-8_4.4x3mm_Pitch0.65mm, symbol 4ms-ic:NJM2068-separate-power
Connections:
- wire segments 334 -> 368
- no-connect marks 11 -> 18
Other:
- note added: "FINDINGS\n-helps to buffer signal on input\n-instead of buffer on 13700, use op amps - get rid of resistor to -V\n-using 100k resistor from 12v through 1M pot to voltage cv input\n *could add voltage divider and use a small pot - seems to need \nto stay within a certain voltage to work….\n-small filtering caps (2x1000pF in series for each side) does a good job getting highhats sometimes\n *need t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"
