File: p1/pcb-dualdrum-dev1.sch (KiCad schematic (older format))
At the start: 156 parts, among them P1 CONN-02x05, U1 082, U2 082, U3 082, U4 082, U5 082, U6 082, U7 082, U8 082-NJM, U9 082

Commit message: wip
Parts:
- gave numbers to parts that had none: 2
Changed lines of the file:
@@
 P 11575 3250
 AR Path="/5B8C674E/5D9AD2ED" Ref="C?"  Part="1"
-AR Path="/5D9AD2ED" Ref="C?"  Part="1"
+AR Path="/5D9AD2ED" Ref="C53"  Part="1"
 AR Path="/5E7668A3/5D9AD2ED" Ref="C?"  Part="1"
-F 0 "C?" V 11525 3300 50  0000 L CNN
+F 0 "C53" V 11525 3300 50  0000 L CNN
 F 1 "1uF" V 11525 2975 50  0000 L CNN
 F 2 "4ms_Capacitor:C_0603" H 11575 3250 50  0001 C CNN
@@
 P 11625 7500
 AR Path="/5B8C674E/5DA4667F" Ref="C?"  Part="1"
-AR Path="/5DA4667F" Ref="C?"  Part="1"
+AR Path="/5DA4667F" Ref="C54"  Part="1"
 AR Path="/5E7668A3/5DA4667F" Ref="C?"  Part="1"
-F 0 "C?" V 11575 7550 50  0000 L CNN
+F 0 "C54" V 11575 7550 50  0000 L CNN
 F 1 "1uF" V 11575 7225 50  0000 L CNN
 F 2 "4ms_Capacitor:C_0603" H 11625 7500 50  0001 C CNN
