File: p1/pcb-dualdrum-dev1.sch (KiCad schematic (older format))
At the start: 156 parts, among them P1 CONN-02x05, U1 082, U2 082, U3 082, U4 082, U5 082, U6 082, U7 082, U8 082-NJM, U9 082

Commit message: looks good - ready to plot
Changed lines of the file:
@@
 EESchema Schematic File Version 4
 LIBS:pcb-dualdrum-dev1-cache
-EELAYER 29 0
+EELAYER 30 0
 EELAYER END
 $Descr A2 23386 16535
@@
 F 5 "Substitution OK" H 1275 2775 50  0001 C CNN "Comments"
 	1    6425 4875
-	0    -1   1    0
+	0    1    1    0
 $EndComp
 NoConn ~ 6575 4875
@@
 F 5 "Substitution OK" H 1325 -1250 50  0001 C CNN "Comments"
 	1    6475 850
-	0    -1   1    0
+	0    1    1    0
 $EndComp
 $EndSCHEMATC
