File: p1/pcb-dualdrum-dev1.kicad_pcb (KiCad board)
At the start: 2 copper layers, 48 x 109.2 mm, 156 parts, among them P1 CONN-02x05, U1 082, U2 082, U3 082, U4 082, U5 082, U6 082, U7 082, U8 082-NJM, U9 082

Commit message: wip
Parts:
- moved R17 0.32 mm to (43.7, -105.4)
Routing:
- net Net-(IN2-Pad3): track 0.00 -> 114.1 mm, vias 0 -> 2
- net Net-(Bypass_2nd_Filter1-Pad1): track 0.00 -> 66.7 mm, vias 0 -> 4
- net Net-(Freq1-Pad2): track 0.00 -> 40.1 mm, vias 0 -> 6
- net Net-(LM1-Pad13): track 0.00 -> 34.2 mm, vias 0 -> 5
- net Net-(LM2-Pad13): track 0.00 -> 32.4 mm, vias 0 -> 5
- net Net-(Bypass_2nd_Filter1-Pad2): track 0.00 -> 29.1 mm, vias 0 -> 3
- net Net-(C10-Pad1): track 0.00 -> 11.7 mm
- net Net-(C5-Pad1): track 0.00 -> 11.6 mm
- net Net-(C4-Pad1): track 0.00 -> 11.6 mm
- net Net-(C9-Pad1): track 0.00 -> 11.1 mm
- net Net-(LM1-Pad14): track 0.00 -> 4.01 mm
- net Net-(LM2-Pad14): track 0.00 -> 3.99 mm
- net Net-(LM1-Pad3): track 0.00 -> 3.83 mm
- net Net-(Freq1-Pad1): track 0.00 -> 3.52 mm
- net Net-(LM2-Pad3): track 0.00 -> 3.49 mm
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
Commit message: about to run drc
Parts:
- moved C18 1.51 mm to (12.7, -24.8)
- moved C42 1.51 mm to (12.5, -28.0)
- moved R45 1.51 mm to (12.5, -21.6)
- moved D2 1.51 mm to (3.30, -21.8)
- moved R36 1.51 mm to (3.48, -28.2)
- moved CD2 1.51 mm to (8.01, -24.9)
- moved C52 1.51 mm to (11.5, -17.7)
- moved R51 1.51 mm to (11.5, -19.2)
- moved C12 1.51 mm to (3.35, -25.0)
- moved R3 0.66 mm to (46.1, -17.5), turned to 90 degrees
Routing:
- net Net-(C17-Pad2): track 1.56 -> 77.2 mm, vias 0 -> 3
- net Net-(C8-Pad2): track 0.00 -> 61.2 mm, vias 0 -> 2
- net Net-(C13-Pad1): track 5.35 -> 35.9 mm, vias 0 -> 1
- net Net-(C12-Pad2): track 0.00 -> 28.4 mm, vias 0 -> 2
- net Net-(C2-Pad2): track 0.00 -> 28.2 mm, vias 0 -> 2
- net Net-(C51-Pad1): track 0.00 -> 27.7 mm, vias 0 -> 2
- net Net-(C13-Pad2): track 9.19 -> 33.7 mm, vias 0 -> 2
- net Net-(IN2-Pad3): track 114.1 -> 135.1 mm, vias 2 -> 4
- net Net-(C7-Pad2): track 0.00 -> 20.8 mm
- net Net-(Bypass_2nd_Filter1-Pad3): track 0.00 -> 19.4 mm, vias 0 -> 1
- net Net-(C11-Pad2): track 0.00 -> 14.3 mm
- net Net-(C1-Pad2): track 0.00 -> 14.0 mm
- net GND: track 533.2 -> 546.9 mm, vias 32 -> 33
- net Net-(C52-Pad1): track 0.00 -> 13.4 mm
- net Net-(C18-Pad2): track 0.00 -> 13.3 mm
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
Commit message: drc cleared - checking for more mistakes
Routing:
- net Net-(Bypass_2nd_Filter2-Pad1): track 81.1 -> 80.1 mm
- net GND: track 546.9 -> 547.8 mm, vias 33 -> 32
- net Net-(R21-Pad1): track 1.88 -> 2.53 mm
- net Net-(R31-Pad1): track 1.86 -> 2.51 mm
Other:
- rule trace_min: 0.2 -> 0
