File: p1/pcb-dualdrum-dev1.kicad_pcb (KiCad board)
At the start: 2 copper layers, 48 x 109.2 mm, 156 parts, among them P1 CONN-02x05, U1 082, U2 082, U3 082, U4 082, U5 082, U6 082, U7 082, U8 082-NJM, U9 082

Commit message: looks good - ready to plot
Connections:
- R1 pad 2: Net-(Freq1-Pad1) -> Net-(Freq1-Pad3)
- R32 pad 2: Net-(Freq2-Pad1) -> Net-(Freq2-Pad3)
Routing:
- net Net-(Freq1-Pad3): track 0.00 -> 16.3 mm, vias 0 -> 1
- net Net-(Freq2-Pad3): track 0.00 -> 8.99 mm, vias 0 -> 1
- net Net-(Freq1-Pad1): track 3.52 -> 0.00 mm
- net Net-(Freq2-Pad1): track 3.30 -> 0.45 mm
- net Net-(CD1-Pad2): track 10.9 -> 11.9 mm
- net Net-(CD2-Pad2): track 10.8 -> 11.7 mm
- net Net-(CD1-Pad11): track 5.86 -> 6.64 mm
Changed lines of the file:
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@@
   (general
     (thickness 1.6)
-    (drawings 4)
-    (tracks 1390)
+    (drawings 12)
+    (tracks 1400)
     (zones 0)
     (modules 156)
@@
     (34 B.Paste user)
     (35 F.Paste user)
-    (36 B.SilkS user)
+    (36 B.SilkS user hide)
     (37 F.SilkS user)
     (38 B.Mask user)
@@
       (net 36 +12V))
     (pad 2 smd rect (at 0.85 0 90) (size 1 1) (layers F.Cu F.Paste F.Mask)
-      (net 76 "Net-(Freq2-Pad1)"))
+      (net 74 "Net-(Freq2-Pad3)"))
     (model Resistors_SMD.3dshapes/R_0603.wrl
       (at (xyz 0 0 0))
@@
       (net 36 +12V))
     (pad 2 smd rect (at 0.85 0 90) (size 1 1) (layers F.Cu F.Paste F.Mask)
-      (net 42 "Net-(Freq1-Pad1)"))
+      (net 40 "Net-(Freq1-Pad3)"))
     (model Resistors_SMD.3dshapes/R_0603.wrl
       (at (xyz 0 0 0))
@@
     )
   )
+  (gr_line (start 6.1976 -89.59088) (end 11.56208 -89.59088) (layer F.SilkS) (width 0.15))
+  (gr_line (start 11.57732 -92.57792) (end 6.1976 -92.57792) (layer F.SilkS) (width 0.15))
+  (gr_line (start 6.1976 -92.52204) (end 6.1976 -89.59088) (layer F.SilkS) (width 0.15))
+  (gr_line (start 11.56208 -89.59088) (end 11.57732 -92.57792) (layer F.SilkS) (width 0.15))
+  (gr_line (start 38.76548 -93.22308) (end 33.38576 -93.22308) (layer F.SilkS) (width 0.15))
+  (gr_line (start 38.75024 -90.23604) (end 38.76548 -93.22308) (layer F.SilkS) (width 0.15))
+  (gr_line (start 33.38576 -90.23604) (end 38.75024 -90.23604) (layer F.SilkS) (width 0.15))
+  (gr_line (start 33.38576 -93.1672) (end 33.38576 -90.23604) (layer F.SilkS) (width 0.15))
   (gr_line (start 0 0) (end 48 0) (layer Edge.Cuts) (width 0.1))
   (gr_line (start 48 0) (end 48 -109.22) (layer Edge.Cuts) (width 0.1))
@@
   (segment (start 36 -87.046) (end 37.7698 -85.2762) (width 0.25) (layer F.Cu) (net 41))
   (segment (start 37.7698 -85.2762) (end 37.7698 -80.5942) (width 0.25) (layer F.Cu) (net 41))
-  (segment (start 44.3749 -87.046) (end 44.4754 -87.1465) (width 0.25) (layer F.Cu) (net 42))
-  (segment (start 41 -87.046) (end 44.3749 -87.046) (width 0.25) (layer F.Cu) (net 42))
+  (segment (start 44.3749 -87.046) (end 44.4754 -87.1465) (width 0.25) (layer F.Cu) (net 40))
+  (via (at 44.44492 -88.36152) (size 0.8) (drill 0.4) (layers F.Cu B.Cu) (net 40))
+  (segment (start 44.4754 -88.33104) (end 44.44492 -88.36152) (width 0.25) (layer F.Cu) (net 40))
+  (segment (start 44.4754 -87.1465) (end 44.4754 -88.33104) (width 0.25) (layer F.Cu) (net 40))
+  (segment (start 33.39756 -89.44356) (end 31 -87.046) (width 0.25) (layer B.Cu) (net 40))
+  (segment (start 43.36288 -89.44356) (end 33.39756 -89.44356) (width 0.25) (layer B.Cu) (net 40))
+  (segment (start 44.44492 -88.36152) (end 43.36288 -89.44356) (width 0.25) (layer B.Cu) (net 40))
   (via (at 37.3761 -12.192) (size 0.8) (drill 0.4) (layers F.Cu B.Cu) (net 43))
   (segment (start 33.8954 -7.4295) (end 33.8954 -8.7113) (width 0.25) (layer F.Cu) (net 43))
@@
   (segment (start 9.5495 -32.99742) (end 9.539837 -32.987757) (width 0.25) (layer F.Cu) (net 72))
   (segment (start 9.5495 -36.4617) (end 9.5495 -32.99742) (width 0.25) (layer F.Cu) (net 72))
+  (via (at 13.97508 -84.82076) (size 0.8) (drill 0.4) (layers F.Cu B.Cu) (net 74))
+  (segment (start 13.98614 -84.8097) (end 13.97508 -84.82076) (width 0.25) (layer F.Cu) (net 74))
+  (segment (start 15.0622 -84.8097) (end 13.98614 -84.8097) (width 0.25) (layer F.Cu) (net 74))
+  (segment (start 9.22524 -84.82076) (end 7 -87.046) (width 0.25) (layer B.Cu) (net 74))
+  (segment (start 13.97508 -84.82076) (end 9.22524 -84.82076) (width 0.25) (layer B.Cu) (net 74))
   (via (at 7.4422 -103.415488) (size 0.8) (drill 0.4) (layers F.Cu B.Cu) (net 75))
   (segment (start 7.4015 -102.4605) (end 7.4015 -103.374788) (width 0.25) (layer F.Cu) (net 75))
@@
   (segment (start 12 -87.046) (end 12 -82.67839) (width 0.25) (layer F.Cu) (net 75))
   (segment (start 16.5485 -87.046) (end 17 -87.046) (width 0.25) (layer F.Cu) (net 76))
-  (segment (start 15.0622 -85.5597) (end 16.5485 -87.046) (width 0.25) (layer F.Cu) (net 76))
-  (segment (start 15.0622 -84.8097) (end 15.0622 -85.5597) (width 0.25) (layer F.Cu) (net 76))
   (segment (start 44.15836 -103.4034) (end 44.139385 -103.4034) (width 0.25) (layer F.Cu) (net 77))
   (segment (start 44.4661 -103.09566) (end 44.15836 -103.4034) (width 0.25) (layer F.Cu) (net 77))
@@
   (segment (start 28.4099 -16.4211) (end 28.4099 -17.1831) (width 0.25) (layer B.Cu) (net 77))
   (segment (start 43.5737 -103.4034) (end 44.139385 -103.4034) (width 0.25) (layer B.Cu) (net 77))
-  (segment (start 39.3079 -21.4299) (end 38.8579 -21.4299) (width 0.25) (layer F.Cu) (net 78))
-  (segment (start 39.932901 -22.054901) (end 39.3079 -21.4299) (width 0.25) (layer F.Cu) (net 78))
-  (segment (start 39.932901 -23.344899) (end 39.932901 -22.054901) (width 0.25) (layer F.Cu) (net 78))
-  (segment (start 39.3079 -23.9699) (end 39.932901 -23.344899) (width 0.25) (layer F.Cu) (net 78))
-  (segment (start 38.8579 -23.9699) (end 39.3079 -23.9699) (width 0.25) (layer F.Cu) (net 78))
   (segment (start 37.2151 -23.9699) (end 37.0332 -23.788) (width 0.25) (layer F.Cu) (net 78))
   (segment (start 38.8579 -23.9699) (end 37.2151 -23.9699) (width 0.25) (layer F.Cu) (net 78))
-  (segment (start 43.8079 -18.8899) (end 44.2579 -18.8899) (width 0.25) (layer F.Cu) (net 79))
-  (segment (start 43.182899 -19.514901) (end 43.8079 -18.8899) (width 0.25) (layer F.Cu) (net 79))
-  (segment (start 43.182899 -20.804899) (end 43.182899 -19.514901) (width 0.25) (layer F.Cu) (net 79))
-  (segment (start 43.8079 -21.4299) (end 43.182899 -20.804899) (width 0.25) (layer F.Cu) (net 79))
-  (segment (start 44.2579 -21.4299) (end 43.8079 -21.4299) (width 0.25) (layer F.Cu) (net 79))
+  (segment (start 40.2082 -21.78812) (end 39.84998 -21.4299) (width 0.25) (layer F.Cu) (net 78))
+  (segment (start 39.84998 -21.4299) (end 38.8579 -21.4299) (width 0.25) (layer F.Cu) (net 78))
+  (segment (start 39.71298 -23.9699) (end 40.2082 -23.47468) (width 0.25) (layer F.Cu) (net 78))
+  (segment (start 40.2082 -23.47468) (end 40.2082 -21.78812) (width 0.25) (layer F.Cu) (net 78))
+  (segment (start 38.8579 -23.9699) (end 39.71298 -23.9699) (width 0.25) (layer F.Cu) (net 78))
   (segment (start 39.3079 -25.2399) (end 38.8579 -25.2399) (width 0.25) (layer F.Cu) (net 79))
   (segment (start 43.1179 -21.4299) (end 39.3079 -25.2399) (width 0.25) (layer F.Cu) (net 79))
   (segment (start 44.2579 -21.4299) (end 43.1179 -21.4299) (width 0.25) (layer F.Cu) (net 79))
+  (segment (start 43.35026 -18.8899) (end 44.2579 -18.8899) (width 0.25) (layer F.Cu) (net 79))
+  (segment (start 42.77868 -19.46148) (end 43.35026 -18.8899) (width 0.25) (layer F.Cu) (net 79))
+  (segment (start 43.18246 -21.4299) (end 42.77868 -21.02612) (width 0.25) (layer F.Cu) (net 79))
+  (segment (start 42.77868 -21.02612) (end 42.77868 -19.46148) (width 0.25) (layer F.Cu) (net 79))
+  (segment (start 44.2579 -21.4299) (end 43.18246 -21.4299) (width 0.25) (layer F.Cu) (net 79))
   (via (at 46.2534 -24.4475) (size 0.8) (drill 0.4) (layers F.Cu B.Cu) (net 80))
   (segment (start 46.2661 -23.4618) (end 46.2661 -24.4348) (width 0.25) (layer F.Cu) (net 80))
@@
   (segment (start 12.3776 -22.3208) (end 12.5222 -22.4654) (width 0.25) (layer F.Cu) (net 81))
   (segment (start 10.7 -22.3208) (end 12.3776 -22.3208) (width 0.25) (layer F.Cu) (net 81))
+  (segment (start 9.0678 -22.953) (end 9.7 -22.3208) (width 0.25) (layer F.Cu) (net 81))
+  (segment (start 9.0678 -24.41956) (end 9.0678 -22.953) (width 0.25) (layer F.Cu) (net 81))
+  (segment (start 9.50904 -24.8608) (end 9.0678 -24.41956) (width 0.25) (layer F.Cu) (net 81))
   (segment (start 9.7 -22.3208) (end 10.7 -22.3208) (width 0.25) (layer F.Cu) (net 81))
-  (segment (start 9.2329 -22.7879) (end 9.7 -22.3208) (width 0.25) (layer F.Cu) (net 81))
-  (segment (start 9.2329 -24.3937) (end 9.2329 -22.7879) (width 0.25) (layer F.Cu) (net 81))
-  (segment (start 10.7 -24.8608) (end 9.7 -24.8608) (width 0.25) (layer F.Cu) (net 81))
-  (segment (start 9.7 -24.8608) (end 9.2329 -24.3937) (width 0.25) (layer F.Cu) (net 81))
+  (segment (start 10.7 -24.8608) (end 9.50904 -24.8608) (width 0.25) (layer F.Cu) (net 81))
   (segment (start 5.75 -24.8608) (end 5.3 -24.8608) (width 0.25) (layer F.Cu) (net 82))
-  (segment (start 6.375001 -25.485801) (end 5.75 -24.8608) (width 0.25) (layer F.Cu) (net 82))
-  (segment (start 6.375001 -27.325799) (end 6.375001 -25.485801) (width 0.25) (layer F.Cu) (net 82))
-  (segment (start 6.3 -27.4008) (end 6.375001 -27.325799) (width 0.25) (layer F.Cu) (net 82))
+  (segment (start 6.45088 -24.8608) (end 5.75 -24.8608) (width 0.25) (layer F.Cu) (net 82))
+  (segment (start 7.01548 -25.4254) (end 6.45088 -24.8608) (width 0.25) (layer F.Cu) (net 82))
+  (segment (start 6.3 -27.4008) (end 7.01548 -26.68532) (width 0.25) (layer F.Cu) (net 82))
+  (segment (start 7.01548 -26.68532) (end 7.01548 -25.4254) (width 0.25) (layer F.Cu) (net 82))
   (segment (start 5.3 -27.4008) (end 6.3 -27.4008) (width 0.25) (layer F.Cu) (net 82))
-  (segment (start 9.56 -21.0508) (end 10.7 -21.0508) (width 0.25) (layer F.Cu) (net 82))
-  (segment (start 5.75 -24.8608) (end 9.56 -21.0508) (width 0.25) (layer F.Cu) (net 82))
+  (segment (start 5.75 -24.8608) (end 6.4574 -24.8608) (width 0.25) (layer F.Cu) (net 82))
+  (segment (start 6.4574 -24.8608) (end 10.2674 -21.0508) (width 0.25) (layer F.Cu) (net 82))
+  (segment (start 10.2674 -21.0508) (end 10.7 -21.0508) (width 0.25) (layer F.Cu) (net 82))
   (segment (start 3.8149 -28.6708) (end 3.4798 -29.0059) (width 0.25) (layer F.Cu) (net 83))
   (segment (start 5.3 -28.6708) (end 3.8149 -28.6708) (width 0.25) (layer F.Cu) (net 83))

Commit message: generated grbs - submitted to pcbcart
Parts:
- added G***: LOGO, 4ms_Symbol:4msLogo_15.5x6.6mm, F.Cu at (23.8, -90.6)
Other:
- board text added: "DEV1"
- board text added: "DUAL DRUM"
