File: p2/dualdrum.sch (KiCad schematic (older format))
At the start: 156 parts, among them P1 CONN-02x05, U1 082, U2 082, U3 082, U4 082, U5 082, U6 082, U7 082, U8 082-NJM, U9 082

Commit message: added notes - made more tests
Other:
- note added: "-changing R23 to 20k prevents \ncircuit from cutting out"
- note added: "cut traces between 13700s\n-freq pot to lm2\n-out put summed together at u6\n\nnow, reconected with jumpers\n-changed r4 and r34 to 100k - seems to help signal on first\nota but the second one still oscillating - so they are back to being\n10ks now -\n\nremoved resistors connecting one shot circuit - need to put them back\ncurrently no filtering cap on R30 - though originally i thought that was \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"
- note added: "fixes \n-cut out issue was due to R23 being to low of value - changed\nfrom 10k to 20k\n\n-filter range caps are currently 1nF - 4.6nF was good - and 10nF was good\nbut too much bass - maybe explore with a range setting switch? hmmmm"
- note removed: "cut traces between 13700s\n-freq pot to lm2\n-out put summed together at u6\n\nnow, reconected with jumpers\n-changed r4 and r34 to 100k - seems to help signal on first\nota but the second one still oscillating \n\nremoved resistors connecting one shot circuit - need to put them back\ncurrently no filtering cap on R30 - though originally i thought that was \nwhat fixed the oscillation\n\nnew prob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"
Changed lines of the file:
@@
 EESchema Schematic File Version 4
-EELAYER 26 0
+LIBS:dualdrum-cache
+EELAYER 30 0
 EELAYER END
 $Descr A2 23386 16535
@@
 100k res to -12v here
 Text Notes 7150 -175 0    50   ~ 0
-cut traces between 13700s\n-freq pot to lm2\n-out put summed together at u6\n\nnow, reconected with jumpers\n-changed r4 and r34 to 100k - seems to help signal on first\nota but the second one still oscillating \n\nremoved resistors connecting one shot circuit - need to put them back\ncurrently no filtering cap on R30 - though originally i thought that was \nwhat fixed the oscillation\n\nnew problem - when setting freq cutoff to highest point, the second\n13700 fails when recieving lower frequencies\n**one theory is harsh edges? may want to try rc filter into 13700\n**another theory may be power draw at lower frequencies? the 2nd 13700\ngoes high when this issue occurs.
+cut traces between 13700s\n-freq pot to lm2\n-out put summed together at u6\n\nnow, reconected with jumpers\n-changed r4 and r34 to 100k - seems to help signal on first\nota but the second one still oscillating - so they are back to being\n10ks now -\n\nremoved resistors connecting one shot circuit - need to put them back\ncurrently no filtering cap on R30 - though originally i thought that was \nwhat fixed the oscillation\n\nnew problem - when setting freq cutoff to highest point, the second\n13700 fails when recieving lower frequencies\n**one theory is harsh edges? may want to try rc filter into 13700\n**another theory may be power draw at lower frequencies? the 2nd 13700\ngoes high when this issue occurs.
 Text Notes 4100 4075 0    50   ~ 0
 adding 100nF  cap in par w/r30 gets rid of oscillation\n*this may not be true\n
+Text Notes 3400 3450 1    50   ~ 0
+-changing R23 to 20k prevents \ncircuit from cutting out
+Text Notes 2825 -350 0    50   ~ 0
+fixes \n-cut out issue was due to R23 being to low of value - changed\nfrom 10k to 20k\n\n-filter range caps are currently 1nF - 4.6nF was good - and 10nF was good\nbut too much bass - maybe explore with a range setting switch? hmmmm
 $EndSCHEMATC
